File: potatoesc.kicad_pcb (KiCad board)
At the start: 2 copper layers, 79 parts, among them J1 Screw_Terminal_01x03, J2 Screw_Terminal_01x05, Q1 BSP89, Q2 BSP89, Q3 BSP89, Q4 BSP89, Q5 BSP89, Q6 BSP89, SW1 SW_Push, U1 TEN20-4811WIN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

Commit message: Added first pcb design
Parts:
- added H6: V_RAW, Connector_Wire:SolderWirePad_1x01_SMD_5x10mm, F.Cu at (126.0, 87.9)
- added H7: V_RAW, Connector_Wire:SolderWirePad_1x01_SMD_5x10mm, F.Cu at (108.1, 87.8)
- added H8: V_RAW, Connector_Wire:SolderWirePad_1x01_SMD_5x10mm, F.Cu at (89.7, 87.8)
- C1, C13, C14, C15, C17, C18, C2, C21, C23, C24, C3, C4, C6, C7: footprint Capacitor_THT:CP_Radial_Tantal_D5.5mm_P5.00mm -> Capacitor_SMD:C_0805_2012Metric_Pad1.18x1.45mm_HandSolder
- C16, C19, C20, C22, C25, C26, C5, C8, C9: footprint Capacitor_THT:CP_Radial_Tantal_D5.5mm_P5.00mm -> Capacitor_SMD:CP_Elec_5x4.4
- Q1, Q2, Q3, Q4, Q5, Q6: footprint Package_TO_SOT_THT:TO-220-3_Vertical -> Package_TO_SOT_THT:TO-220-3_Horizontal_TabDown
- R1, R10, R11, R12, R13, R14, R15, R16, R17, R18, R19, R2, R20, R21, R22, R3, R4, R5, R6, R7, R8, R9: footprint Resistor_THT:R_Axial_DIN0411_L9.9mm_D3.6mm_P15.24mm_Horizontal -> Resistor_SMD:R_1206_3216Metric_Pad1.30x1.75mm_HandSolder
- moved C21 202.1 mm to (78.2, 120.5), turned to 0 degrees
- moved C22 193.2 mm to (79.4, 127.5), turned to 0 degrees
- moved D4 181.5 mm to (72.5, 134.7), turned to 180 degrees
- moved C15 177.1 mm to (104.4, 121.0), turned to 0 degrees
- moved C23 177.0 mm to (88.1, 133.2), turned to 0 degrees
- moved C16 163.8 mm to (110.5, 127.4), turned to 0 degrees
- moved C24 160.1 mm to (96.8, 133.2), turned to 180 degrees
- moved C25 158.2 mm to (89.2, 127.5), turned to 0 degrees
- moved C4 153.6 mm to (129.8, 120.8), turned to 0 degrees
- moved D3 150.0 mm to (108.7, 134.4), turned to 180 degrees
- moved C17 147.7 mm to (119.6, 132.3), turned to 0 degrees
- moved C26 139.6 mm to (99.5, 127.4), turned to 180 degrees
- moved C5 136.5 mm to (140.7, 127.4), turned to 0 degrees
- moved C19 129.4 mm to (120.2, 127.4), turned to 0 degrees
- moved C18 128.4 mm to (131.1, 132.2), turned to 180 degrees
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Routing:
- net +12V: track 0.00 -> 302.5 mm
- net CTRL_CL: track 0.00 -> 107.9 mm
- net CTRL_CH: track 0.00 -> 103.2 mm
- net COM_A: track 0.00 -> 89.5 mm
- net V_RAW: track 0.00 -> 86.4 mm
- net CTRL_BL: track 0.00 -> 85.3 mm
- net CTRL_BH: track 0.00 -> 80.5 mm
- net Net-(Q3-G): track 0.00 -> 79.7 mm, vias 0 -> 1
- net COM_B: track 0.00 -> 77.9 mm
- net Net-(Q2-G): track 0.00 -> 70.1 mm, vias 0 -> 1
- net COM_C: track 0.00 -> 67.2 mm
- net CTRL_AL: track 0.00 -> 66.3 mm
- net DRV_BL: track 0.00 -> 63.4 mm
- net CTRL_AH: track 0.00 -> 61.4 mm
- net DRV_AL: track 0.00 -> 60.3 mm
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- added copper zone on B.Cu, net GND
- added copper zone on F.Cu, net GND
- added copper zone on F.Cu, net Net-(F1-Pad1)
- added copper zone on F.Cu, net V_RAW
Other:
- board outline added: 200.2 x 98.8 mm
